File: Mentor.kicad_pcb (KiCad board)
At the start: 2 copper layers, 50 x 100 mm, 41 parts, among them J1 CONN_01X02, J2 CONN_01X06, J3 CONN_01X09, J4 CONN_01X10, J5 CONN_01X02, J6 CONN_01X03, J7 CONN_01X09, Q1 PZT2222A, Q2 PZT2222A, Q3 IRFR3303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

Commit message: upgrade to kicad 5.x
Parts:
- moved C4 118.3 mm to (61.8, 106.4)
- moved BZ1 118.3 mm to (82.0, 39.0)
- moved C1 118.3 mm to (51.6, 105.4)
- moved C2 118.3 mm to (68.0, 111.5)
- moved C3 118.3 mm to (71.5, 112.5)
- moved C5 118.3 mm to (67.5, 103.5)
- moved C6 118.3 mm to (67.5, 46.5)
- moved D1 118.3 mm to (61.0, 64.5)
- moved J1 118.3 mm to (47.0, 111.0)
- moved J2 118.3 mm to (47.0, 72.0)
- moved J3 118.3 mm to (87.5, 60.5)
- moved J4 118.3 mm to (47.0, 94.0)
- moved J5 118.3 mm to (87.5, 99.0)
- moved J6 118.3 mm to (87.5, 106.0)
- moved J7 118.3 mm to (87.5, 84.0)
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Routing:
- net GND: track 371.5 -> 187.2 mm, vias 79 -> 281
Other:
- board text added: "Mentor Μέντωρ V2.0 ON7EQ SSPA control board Drawing f6itu"
- board text removed: "Mentor Μέντωρ V2.0 ON7EQ SSPA control board routing by f6itu"
