File: Mentor.sch (KiCad schematic (older format))
At the start: 41 parts, among them J1 CONN_01X02, J2 CONN_01X06, J3 CONN_01X09, J4 CONN_01X10, J5 CONN_01X02, J6 CONN_01X03, J7 CONN_01X09, Q1 PZT2222A, Q2 PZT2222A, Q3 IRFR3303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

Commit message: Mentor V3.0 W6PQL compatible
Parts:
- added J8: Conn_01x05, conn_kk100:kk100_22-23-2051, symbol Connector_Generic:Conn_01x05
- added R10: 5k, Resistor_SMD:R_0805_2012Metric_Pad1.15x1.40mm_HandSolder, symbol Device:R
- added R11, R14, R15: 1k5, Resistor_SMD:R_0805_2012Metric_Pad1.15x1.40mm_HandSolder, symbol Device:R
- added R12: 3k3, Resistor_SMD:R_0805_2012Metric_Pad1.15x1.40mm_HandSolder, symbol Device:R
- added R13: 2k, Resistor_SMD:R_0805_2012Metric_Pad1.15x1.40mm_HandSolder, symbol Device:R
- added R16, R17: 500R, Resistor_SMD:R_0805_2012Metric_Pad1.15x1.40mm_HandSolder, symbol Device:R
- added RV2, RV3: 2k, Trimmer_3314G1_Handsoldering:Trimmer_3314G1_Handsoldering, symbol Device:R_POT
- BZ1: footprint Buzzers_Beepers:Buzzer_12x9.5RM7.6 -> Buzzer_Beeper:Buzzer_12x9.5RM7.6; symbol Buzzer -> Mentor-rescue:Buzzer
- C1, C3, C5: footprint Capacitors_SMD:C_0805_HandSoldering -> Capacitor_SMD:C_0805_2012Metric_Pad1.15x1.40mm_HandSolder; symbol C_Small -> Mentor-rescue:C_Small
- C2: footprint Capacitors_Tantalum_SMD:CP_Tantalum_Case-C_EIA-6032-28_Hand -> Capacitor_Tantalum_SMD:CP_EIA-6032-28_Kemet-C_Pad2.25x2.35mm_HandSolder; symbol CP1_Small -> Mentor-rescue:CP1_Small
- C4: footprint Capacitors_SMD:C_0805_HandSoldering -> Capacitor_SMD:C_0805_2012Metric_Pad1.15x1.40mm_HandSolder; symbol CP1_Small -> Mentor-rescue:CP1_Small
- C6: footprint Capacitors_SMD:C_0805_HandSoldering -> Capacitor_SMD:C_0805_2012Metric_Pad1.15x1.40mm_HandSolder; symbol C -> Mentor-rescue:C
- D1: footprint Diodes_SMD:D_0805 -> Diode_SMD:D_0805_2012Metric_Pad1.15x1.40mm_HandSolder; symbol LED -> Mentor-rescue:LED
- J1, J5: symbol CONN_01X02 -> Mentor-rescue:CONN_01X02
- J2: symbol CONN_01X06 -> Mentor-rescue:CONN_01X06
- J3, J7: symbol CONN_01X09 -> Mentor-rescue:CONN_01X09
- J4: symbol CONN_01X10 -> Mentor-rescue:CONN_01X10
- J6: symbol CONN_01X03 -> Mentor-rescue:CONN_01X03
- L1, L2, L3, L4, L5, L6: symbol L_cap -> l_cap:L_cap
- Q1, Q2: footprint TO_SOT_Packages_SMD:SOT-223 -> Package_TO_SOT_SMD:SOT-223; symbol PZT2222A -> Mentor-rescue:PZT2222A
- Q3: footprint TO_SOT_Packages_SMD:TO-252-3_TabPin2 -> Package_TO_SOT_SMD:TO-252-3_TabPin2; symbol IRF3205 -> Mentor-rescue:IRF3205
- R1, R2, R3, R4, R5, R6, R7, R8, R9: footprint Resistors_SMD:R_0805_HandSoldering -> Resistor_SMD:R_0805_2012Metric_Pad1.15x1.40mm_HandSolder; symbol R -> Mentor-rescue:R
- RL1: symbol EC2-5NU -> ee2-5nu:EC2-5NU
- RV1: symbol POT -> Mentor-rescue:POT
- TP1, TP2, TP3, TP4: symbol TEST -> Mentor-rescue:TEST
- U1: footprint TO_SOT_Packages_SMD:TO-252-3_TabPin2 -> Package_TO_SOT_SMD:TO-252-3_TabPin2; symbol KA78M05_TO252 -> Mentor-rescue:KA78M05_TO252
- U2: symbol Arduino_Nano -> arduino_nano:Arduino_Nano
Connections:
- net +5V: now also U2.12 (5V); no longer U2.15 (Vin)
- net GND: now also J8.3 (Pin_3), R15.1, RV2.1, RV3.1
- net at R3.1, U2.10 (A6): now also R14.1, R17.2
- net at U2.17 ((RX)D0): now also J8.4 (Pin_4)
- net at U2.20 ((int2)D2): now also R12.1, R15.2
- net at R2.1, U2.9 (A5): now also R13.1, R16.2
- new net: R10.1, R13.2
- new net: J8.1 (Pin_1), R10.2
- new net: R16.1, RV2.2, RV2.3
- new net: J8.2 (Pin_2), R11.2
- new net: J8.5 (Pin_5), R12.2
- new net: R11.1, R14.2
- new net: R17.1, RV3.2, RV3.3
- no-connect marks 15 -> 13
Other:
- note added: "13.8V sense"
- note added: "24V Sense"
- note added: "3.0\n"
- note added: "Bypass/Operate\n"
- note added: "If 12 & 24V Sense is in use, \ndo not install R2 and R3"
- note added: "J8 and associated components \nfor W6PQL board only. \nIt should not be installed/wired\nfor Alex frontend"
- note added: "May24th 2017 updated 29/04/2020\n"
- note added: "Mentor\nA power/U/I/VSWR/Temp. indicator\nand security system\nBy ON7EQ\nfor the Hermes SDR familly and W6PQL control board"
- note added: "Reset/Alarm"
- note removed: "May24th 2017"
- note removed: "Mentor\nA power/U/I/VSWR/Temp. indicator\nand security system\nBy ON7EQ\nfor the Hermes SDR familly"
- moved on the sheet: R2, R3
